File: Micro5V3A.kicad_pcb (KiCad board)
At the start: 2 copper layers, 23.4 x 15.1 mm, 16 parts, among them J1 EnablePin, J2 5V, J3 GND, J4 VIN, J5 GND, U1 TPS563209

Commit message: slight edit
Routing:
- net Net-(C3-Pad2): vias 11 -> 12
Changed lines of the file:
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@@
     (thickness 1.6)
     (drawings 12)
-    (tracks 55)
+    (tracks 56)
     (zones 0)
     (modules 16)
@@
   (gr_line (start 131.191 39.878) (end 131.191 54.991) (layer Edge.Cuts) (width 0.2))
   (gr_line (start 154.559 39.878) (end 131.191 39.878) (layer Edge.Cuts) (width 0.2))
-  (via (at 137.287 47.625) (size 1) (drill 0.4) (layers F.Cu B.Cu) (net 6))
-  (via (at 138.938 47.625) (size 1) (drill 0.4) (layers F.Cu B.Cu) (net 6))
-  (via (at 138.176 48.641) (size 1) (drill 0.4) (layers F.Cu B.Cu) (net 6))
-  (via (at 139.827 48.641) (size 1) (drill 0.4) (layers F.Cu B.Cu) (net 6))
   (segment (start 146.49 49.53) (end 145.71 49.53) (width 0.25) (layer F.Cu) (net 1))
   (segment (start 149.225 52.324) (end 148.20849 51.30749) (width 0.25) (layer F.Cu) (net 1))
@@
   (via (at 136.525 44.704) (size 1) (drill 0.4) (layers F.Cu B.Cu) (net 5))
   (via (at 136.525 46.101) (size 1) (drill 0.4) (layers F.Cu B.Cu) (net 5))
+  (via (at 137.287 47.625) (size 1) (drill 0.4) (layers F.Cu B.Cu) (net 6))
+  (via (at 138.938 47.625) (size 1) (drill 0.4) (layers F.Cu B.Cu) (net 6))
+  (via (at 138.176 48.641) (size 1) (drill 0.4) (layers F.Cu B.Cu) (net 6))
+  (via (at 139.827 48.641) (size 1) (drill 0.4) (layers F.Cu B.Cu) (net 6))
   (segment (start 148.971 48.641) (end 148.971 48.066) (width 0.25) (layer F.Cu) (net 6))
   (via (at 148.971 47.371) (size 1) (drill 0.4) (layers F.Cu B.Cu) (net 6))
@@
   (segment (start 143.891 47.371) (end 142.367 47.371) (width 0.25) (layer B.Cu) (net 6))
   (via (at 136.652 48.641) (size 1) (drill 0.4) (layers F.Cu B.Cu) (net 6))
+  (via (at 142.367 49.403) (size 1) (drill 0.4) (layers F.Cu B.Cu) (net 6))
   (via (at 135.001 51.562) (size 1) (drill 0.4) (layers F.Cu B.Cu) (net 7))
   (via (at 135.001 52.959) (size 1) (drill 0.4) (layers F.Cu B.Cu) (net 7))
